Commit message: update lwa geometry

File: schunk_description/urdf/lwa/lwa.urdf.xacro (robot description, xacro)
@@ -99,5 +99,5 @@
 		<!-- joint between arm_2_link and arm_3_link -->
 		<joint name="${name}_3_joint" type="revolute">
-			<origin xyz="0 -0.408 0" rpy="-1.5708 0 0"/>
+			<origin xyz="0 -0.328 0" rpy="-1.5708 0 0"/>
 			<parent link="${name}_2_link"/>
 			<child link="${name}_3_link"/>
@@ -163,5 +163,5 @@
 		<!-- joint between arm_4_link and arm_5_link -->
 		<joint name="${name}_5_joint" type="revolute">
-			<origin xyz="0 -0.3165 0" rpy="-1.5708 0 0" />
+			<origin xyz="0 -0.2765 0" rpy="-1.5708 0 0" />
 			<parent link="${name}_4_link"/>
 			<child link="${name}_5_link"/>
