Commit message: Corrected urdf, now with the right lwa_extended measurement

File: schunk_description/urdf/lwa_extended/lwa_extended.urdf.xacro (robot description, xacro)
@@ -99,5 +99,5 @@
 		<!-- joint between arm_2_link and arm_3_link -->
 		<joint name="${name}_3_joint" type="revolute">
-			<origin xyz="0 -0.328 0" rpy="-1.5708 0 0"/>
+			<origin xyz="0 -0.403 0" rpy="-1.5708 0 0"/>
 			<parent link="${name}_2_link"/>
 			<child link="${name}_3_link"/>
@@ -163,5 +163,5 @@
 		<!-- joint between arm_4_link and arm_5_link -->
 		<joint name="${name}_5_joint" type="revolute">
-			<origin xyz="0 -0.2765 0" rpy="-1.5708 0 0" />
+			<origin xyz="0 -0.3265 0" rpy="-1.5708 0 0" />
 			<parent link="${name}_4_link"/>
 			<child link="${name}_5_link"/>

Commit message: update lwa extended geometry

File: schunk_description/urdf/lwa_extended/lwa_extended.urdf.xacro (robot description, xacro)
@@ -225,5 +225,5 @@
 		<!-- joint between arm_6_link and arm_7_link -->
 		<joint name="${name}_7_joint" type="revolute">
-			<origin xyz="0 -0.237448 0" rpy="-1.5708 0 0" />
+			<origin xyz="0 -0.1927 0" rpy="-1.5708 0 0" />
 			<parent link="${name}_6_link"/>
 			<child link="${name}_7_link"/>
